File: pm25.sch (EAGLE design)
At the start: 36 parts, among them J1 CON-0024, Q1 TRANSISTOR-NPN-40V-0.2A-SOT23, Q2 TR-0001, U1 POWER-VREG-FB-EN-SW-350MA, U2 CCS811B-JOPD500, U3 POWER-SWITCH-SIP32509DT, U4 SI7021-A20-GM1R

Commit message: remove dust sensor and other extra circuitry
Parts:
- removed C3: 4.7u, wolff-den:CAP-0010
- removed C5: 10u, wolff-den:CAP-10U-6.3V-0603
- removed J1: CON-0024, wolff-den:CON-0024
- removed JP2: (no value), microbuilder:HEADER-1X12
- removed JP4: (no value), microbuilder:HEADER-1X16ROUND
- removed L1: 4.7u, wolff-den:IND-0003
- removed L2: 2k, wolff-den:FERRITE-0805
- removed PCB1: PCB-PS-CCS811-SI7021, wolff-den:PCB-PS-CCS811-SI7021
- removed Q1: TRANSISTOR-NPN-40V-0.2A-SOT23, wolff-den:TRANSISTOR-NPN-40V-0.2A-SOT23
- removed Q2: TR-0001, wolff-den:TR-0001
- removed R1, R10, R11, R7: 100k, wolff-den:RES-0041
- removed R12: 1k, wolff-den:RES-0039
- removed R13: 976k, wolff-den:RES-976K-1%-0402
- removed R8: 309k, wolff-den:RES-309K-1%-0402
- removed TP1: TP, wolff-den:TP
- removed U$31, U$32: MOUNTINGHOLE2.5, microbuilder:MOUNTINGHOLE2.5
- removed U$34, U$35: FIDUCIAL"", microbuilder:FIDUCIAL""
- removed U1: POWER-VREG-FB-EN-SW-350MA, wolff-den:POWER-VREG-FB-EN-SW-350MA
- removed U3: POWER-SWITCH-SIP32509DT, wolff-den:POWER-SWITCH-SIP32509DT
Connections:
- removed net N$1: L1.1, U1.SW
- removed net N$2: R13.1, R8.2, U1.VFB
- removed net N$3: Q1.E, R11.2, U3.EN
- removed net N$6: Q2.D, R10.1, U1.EN
- removed net N$7: Q1.B, R12.2
- removed net V5V0_BEAD: C5.1, L2.1, R13.2, U1.VOUT, U3.VOUT
- removed net V5V0_HAT: J1.P$2, L2.2, TP1.TP
- net !RESET: no longer JP4.16
- net +3V3: no longer JP4.15
- net A0: no longer JP4.12
- net A1: no longer JP4.11
- net A2: no longer JP4.10
- net A3: no longer JP4.9
- net A4: no longer JP4.8
- net A5: no longer JP4.7
- net D2: no longer JP2.10
- net D3: no longer JP2.9
- net D4: no longer JP2.8
- net D5: no longer JP2.7, R10.2, R12.1, R7.2
- net D6: no longer JP2.6
- net D7: no longer JP2.5
- net D8: no longer JP2.4
- net EN: no longer JP2.2
- net GND: no longer C3.2, C5.2, J1.P$8, JP4.13, Q2.S, R1.1, R11.1, R7.1, R8.1, U1.GND, U3.GND
- net MD: no longer JP4.14
- net MISO: no longer JP4.4
- net MOSI: no longer JP4.5
- net NC: no longer JP4.1
- net RX: no longer J1.P$6, JP4.3
- net SCK: no longer JP4.6
- net SCL: no longer JP2.11
- net SDA: no longer JP2.12
- net TX: no longer J1.P$7, JP4.2
- net VBAT: no longer C3.1, JP2.1, L1.2, U1.VIN
- net VBUS: no longer JP2.3, Q1.C, Q2.G, R1.2, U3.VIN
Other:
- note removed: "Boost"
- note removed: "HPMA115 Connection"
- note removed: "Power if plugged in"

Commit message: rename the parts sequentially
Parts:
- removed R9: 100k, wolff-den:RES-0041
- removed U4: SI7021-A20-GM1R, wolff-den:SI7021-A20-GM1R
- added R1: 20k, wolff-den:RES-0054
- added U1: CCS811B-JOPD500, wolff-den:CCS811B-JOPD500
- R2: value 100k -> 20k; device wolff-den:RES-0041 -> wolff-den:RES-0054
- R4, R5: value 20k -> 100k; device wolff-den:RES-0054 -> wolff-den:RES-0041
- U2: value CCS811B-JOPD500 -> SI7021-A20-GM1R; device wolff-den:CCS811B-JOPD500 -> wolff-den:SI7021-A20-GM1R
- renumbered JP3 to JP2
Connections:
- net +3V3: now also R1.2, U1.VDD, U2.VCC; no longer R5.2, U2.VDD, U4.VCC
- net D5: now also R6.1, U1.!RESET; no longer R2.1, U2.!RESET
- net D6: now also U1.!WAKE; no longer U2.!WAKE
- net D8: now also R4.1, U1.!INT; no longer R6.1, U2.!INT
- net GND: now also R5.1, U1.EP_GND, U2.GND; no longer R9.1, U2.EP_GND, U4.GND
- net N$4: now also R5.2, U1.ADDR; no longer R9.2, U2.ADDR
- net N$5: now also U1.PWM, U1.SENSE; no longer U2.PWM, U2.SENSE
- net SCL: now also R2.1, U1.SCL; no longer R4.1, U4.SCL
- net SDA: now also R1.1, U1.SDA; no longer R5.1, U4.SDA
Other:
- moved on the sheet: C1, C2, R2, R4, R5, R6
